File: 1_Documentacao/2_Hardware/06_All_in_One_Boards_V1.0/All_in_One_Boards_V1.0.brd (EAGLE design)
At the start: 140 x 220 mm, 132 parts

Commit message: Update All in One Boards
Other:
- board size 140 x 220 mm -> 153.8 x 220 mm
Changed lines of the file:
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@@
 <setting verticaltext="up"/>
 </settings>
-<grid distance="0.1" unitdist="mm" unit="mm" style="lines" multiple="1" display="yes" altdistance="5" altunitdist="mil" altunit="mil"/>
+<grid distance="0.25" unitdist="mm" unit="mm" style="lines" multiple="1" display="yes" altdistance="5" altunitdist="mil" altunit="mil"/>
 <layers>
 <layer number="1" name="Top" color="4" fill="1" visible="yes" active="yes"/>
@@
 <text x="145.255" y="13.325" size="1.4224" layer="21" rot="R90">V1.0</text>
 <text x="-5.755" y="92.575" size="1.4224" layer="21" rot="R270">V1.0</text>
+<wire x1="0" y1="0" x2="-6.75" y2="0" width="0.1524" layer="20"/>
+<wire x1="-6.75" y1="0" x2="-6.75" y2="220" width="0.1524" layer="20"/>
+<wire x1="-6.75" y1="220" x2="140" y2="220" width="0.1524" layer="20"/>
+<wire x1="140" y1="220" x2="147" y2="220" width="0.1524" layer="20"/>
+<wire x1="147" y1="220" x2="147" y2="0" width="0.1524" layer="20"/>
+<wire x1="147" y1="0" x2="0" y2="0" width="0.1524" layer="20"/>
 </plain>
 <attributes>
