File: 1_Documentacao/2_Hardware/10_All_in_One_Board_V2.0/All_in_One_Boards_V2.0.brd (EAGLE design)
At the start: 140 x 220 mm, 135 parts

Commit message: Update All in One Boards
Parts:
- added 4K3: (no value), rcl:0207/10
- added ESP8266D1MINI2: (no value), esp8266modules:WEMOS-D1-MINI_SEM_LAYOUT
- added RJ2: ALI-RJ45_SEM_LAYOUT, AliExpressRJ45:ALI-RJ45_SEM_LAYOUT
- added SJ28: (no value), jumper:SJ
- added U$67: MCP2515_MODULE_SEM_LAYOUT, MCP2515_Module:MCP2515_MODULE_SEM_LAYOUT
- added U$68, U$69, U$70, U$71, U$72, U$73, U$74, U$75, U$76, U$77, U$78, U$79, U$80, U$81, U$82, U$83, U$84, U$85: TP, edurobotParts:TP
Connections:
- new net GND3: ESP8266D1MINI2.GND, RJ2.1, RJ2.2, RJ2.P$1, RJ2.P$2, U$67.GND, U$82.P$1
- new net N$138: RJ2.3, U$75.P$1
- new net N$139: RJ2.7, U$84.P$1
- new net N$140: RJ2.8, U$85.P$1
- new net N$141: ESP8266D1MINI2.RESET, U$68.P$1
- new net N$142: ESP8266D1MINI2.A0, U$69.P$1
- new net N$143: ESP8266D1MINI2.D0, U$70.P$1
- new net N$144: ESP8266D1MINI2.D5, U$67.SCK, U$71.P$1
- new net N$145: 4K3.2, ESP8266D1MINI2.D6, SJ28.2, U$72.P$1
- new net N$146: ESP8266D1MINI2.D7, U$67.MOSI, U$73.P$1
- new net N$147: ESP8266D1MINI2.D8, U$67.CS, U$74.P$1
- new net N$148: ESP8266D1MINI2.D4, U$81.P$1
- new net N$149: ESP8266D1MINI2.D3, U$80.P$1
- new net N$150: ESP8266D1MINI2.D2, U$79.P$1
- new net N$151: ESP8266D1MINI2.D1, U$78.P$1
- new net N$152: ESP8266D1MINI2.RX, U$77.P$1
- new net N$153: ESP8266D1MINI2.TX, U$76.P$1
- new net N$154: ESP8266D1MINI2.5V, RJ2.4, U$67.VCC, U$83.P$1
- new net N$155: RJ2.5, U$67.CL
- new net N$156: RJ2.6, U$67.CH
- new net N$157: 4K3.1, SJ28.1, U$67.MISO
Routing:
- net N$154: track 0.00 -> 61.3 mm, vias 0 -> 2
- net N$144: track 0.00 -> 52.9 mm, vias 0 -> 1
- net N$138: track 0.00 -> 51.9 mm
- net N$146: track 0.00 -> 51.8 mm, vias 0 -> 1
- net N$147: track 0.00 -> 44.0 mm
- net N$145: track 0.00 -> 32.2 mm
- net N$157: track 0.00 -> 24.1 mm, vias 0 -> 1
- net N$140: track 0.00 -> 23.1 mm
- net N$156: track 0.00 -> 21.0 mm
- net N$139: track 0.00 -> 19.8 mm
- net N$155: track 0.00 -> 16.0 mm
- net N$148: track 0.00 -> 6.79 mm
- net N$152: track 0.00 -> 6.79 mm
- net N$151: track 0.00 -> 6.79 mm
- net N$153: track 0.00 -> 6.79 mm
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- added copper zone on layer 1, net GND3
- added copper zone on layer 16, net GND3
Other:
- outline, holes or cut-outs redrawn
